Commit message: added second gps

File: models/basic_mobile_bot_v1.urdf (robot description, URDF)
Before this commit: robot basic_mobile_bot, 5 links, 4 joints
Links:
- added link gps2_link
Joints:
- added joint gps2_joint: type fixed, parent base_link, child gps2_link, origin xyz=0.10 0 0.05 rpy=0 0 0
